File: electronics/electronics.kicad_sch (KiCad schematic)
At the start: 4 parts, among them J1 Conn_01x06, SW1 Button

Commit message: Added servo
Parts:
- added M1: Motor_Servo, symbol Motor:Motor_Servo
Connections:
- net +5V: now also M1.2 (+)
- net GND: now also M1.3 (-)
- net at A1.13 (D10): now also M1.1 (PWM)
Changed lines of the file:
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@@
   (junction (at 110.49 93.98) (diameter 0) (color 0 0 0 0)
   )
+  (junction (at 110.49 120.65) (diameter 0) (color 0 0 0 0)
+  )
   (wire (pts (xy 105.41 88.9) (xy 105.41 76.2))
     (stroke (width 0) (type default))
@@
     (stroke (width 0) (type default))
   )
+  (wire (pts (xy 104.14 110.49) (xy 104.14 109.22))
+    (stroke (width 0) (type default))
+  )
   (wire (pts (xy 102.87 86.36) (xy 102.87 81.28))
     (stroke (width 0) (type default))
   )
+  (wire (pts (xy 100.33 110.49) (xy 104.14 110.49))
+    (stroke (width 0) (type default))
+  )
   (wire (pts (xy 120.65 88.9) (xy 127 88.9))
     (stroke (width 0) (type default))
@@
     (stroke (width 0) (type default))
   )
+  (wire (pts (xy 95.25 106.68) (xy 100.33 106.68))
+    (stroke (width 0) (type default))
+  )
   (wire (pts (xy 110.49 93.98) (xy 110.49 104.14))
     (stroke (width 0) (type default))
@@
     (stroke (width 0) (type default))
   )
+  (wire (pts (xy 99.06 104.14) (xy 99.06 101.6))
+    (stroke (width 0) (type default))
+  )
   (wire (pts (xy 130.81 120.65) (xy 130.81 124.46))
     (stroke (width 0) (type default))
@@
     (stroke (width 0) (type default))
   )
+  (wire (pts (xy 97.79 120.65) (xy 110.49 120.65))
+    (stroke (width 0) (type default))
+  )
   (wire (pts (xy 130.81 120.65) (xy 139.7 120.65))
     (stroke (width 0) (type default))
   )
+  (wire (pts (xy 95.25 109.22) (xy 97.79 109.22))
+    (stroke (width 0) (type default))
+  )
   (wire (pts (xy 107.95 78.74) (xy 127 78.74))
     (stroke (width 0) (type default))
@@
     (stroke (width 0) (type default))
   )
+  (wire (pts (xy 100.33 106.68) (xy 100.33 110.49))
+    (stroke (width 0) (type default))
+  )
   (wire (pts (xy 121.92 86.36) (xy 127 86.36))
     (stroke (width 0) (type default))
   )
+  (wire (pts (xy 95.25 104.14) (xy 99.06 104.14))
+    (stroke (width 0) (type default))
+  )
   (wire (pts (xy 142.24 60.96) (xy 142.24 66.04))
     (stroke (width 0) (type default))
   )
+  (wire (pts (xy 99.06 101.6) (xy 127 101.6))
+    (stroke (width 0) (type default))
+  )
   (wire (pts (xy 107.95 91.44) (xy 107.95 78.74))
     (stroke (width 0) (type default))
   )
   (wire (pts (xy 120.65 104.14) (xy 127 104.14))
+    (stroke (width 0) (type default))
+  )
+  (wire (pts (xy 97.79 109.22) (xy 97.79 120.65))
     (stroke (width 0) (type default))
   )
@@
         )
       )
+    )
+  )
+  (symbol (lib_id "Motor:Motor_Servo") (at 87.63 106.68 0) (mirror y) (unit 1)
+    (in_bom yes) (on_board yes) (dnp no)
+    (property "Reference" "M1" (at 86.3711 115.57 0)
+      (effects (font (size 1.27 1.27)))
+    )
+    (property "Value" "Motor_Servo" (at 86.3711 113.03 0)
+      (effects (font (size 1.27 1.27)))
+    )
+    (property "Footprint" "" (at 87.63 111.506 0)
+      (effects (font (size 1.27 1.27)) hide)
+    )
+    (property "Datasheet" "http://forums.parallax.com/uploads/attachments/46831/74481.png" (at 87.63 111.506 0)
+      (effects (font (size 1.27 1.27)) hide)
+    )
+    (pin "1")
+    (pin "2")
+    (pin "3")
+    (instances
+      (project "electronics"
+        (path "/aed23a6e-b4a8-42aa-8962-301c537d02dc"
+          (reference "M1") (unit 1)
+        )
+      )
+    )
+  )
+  (symbol (lib_id "power:+5V") (at 104.14 109.22 0) (unit 1)
+    (in_bom yes) (on_board yes) (dnp no) (fields_autoplaced)
+    (property "Reference" "#PWR03" (at 104.14 113.03 0)
+      (effects (font (size 1.27 1.27)) hide)
+    )
+    (property "Value" "+5V" (at 104.14 104.14 0)
+      (effects (font (size 1.27 1.27)))
+    )
+    (property "Footprint" "" (at 104.14 109.22 0)
+      (effects (font (size 1.27 1.27)) hide)
+    )
+    (property "Datasheet" "" (at 104.14 109.22 0)
+      (effects (font (size 1.27 1.27)) hide)
+    )
+    (pin "1")
+    (instances
+      (project "electronics"
+        (path "/aed23a6e-b4a8-42aa-8962-301c537d02dc"
+          (reference "#PWR03") (unit 1)
+        )
+      )
